Commit message: So changes to fix error

File: description/lidar.xacro (robot description, xacro)
@@ -11,5 +11,5 @@
             <geometry>
                 <!-- <cylinder radius="0.05" length="0.04"/> -->
-                <mesh filename="file://$(find test_bot)/meshes/Rplidar.stl" scale="0.001 0.001 0.001" />
+                <mesh filename="file://$(find slam_bot)/meshes/Rplidar.stl" scale="0.001 0.001 0.001" />
             </geometry>
             <material name="black"/>
@@ -18,5 +18,5 @@
             <geometry>
                 <!-- <cylinder radius="0.05" length="0.04"/> -->
-                <mesh filename="file://$(find test_bot)/meshes/Rplidar.stl" scale="0.001 0.001 0.001" />
+                <mesh filename="file://$(find slam_bot)/meshes/Rplidar.stl" scale="0.001 0.001 0.001" />
             </geometry>
         </collision>

File: description/robot_core.xacro (robot description, xacro)
@@ -41,6 +41,6 @@
             <origin xyz="0.08 0 0"/>
             <geometry>
-                <mesh filename="file://$(find test_bot)/meshes/Chassis.stl" scale="0.001 0.001 0.001" />
-                <!-- <mesh filename="$(find test_bot)/stl/Chassis.stl" scale="0.001 0.001 0.001" /> -->
+                <mesh filename="file://$(find slam_bot)/meshes/Chassis.stl" scale="0.001 0.001 0.001" />
+                <!-- <mesh filename="$(find slam_bot)/stl/Chassis.stl" scale="0.001 0.001 0.001" /> -->
             </geometry>
             <material name="black"/>
