Commit message: Added exploration and adjusted some files

File: description/camera.xacro (robot description, xacro)
@@ -4,5 +4,5 @@
         <parent link="chassis"/>
         <child link="camera_link"/>
-        <origin xyz="0.305 0 0.08" rpy="0 0 0"/>
+        <origin xyz="0.150 0 0.08" rpy="0 0 0"/>
     </joint>
     <link name="camera_link">
@@ -11,5 +11,5 @@
                 <box size="0.010 0.03 0.03"/>
             </geometry>
-            <material name="red"/>
+            <material name="green"/>
         </visual>
     </link>
@@ -21,5 +21,5 @@
     <link name="camera_link_optical"></link>
     <gazebo reference="camera_link">
-        <material>Gazebo/Red</material>
+        <material>Gazebo/Green</material>
         <sensor name="camera" type="camera">
             <pose> 0 0 0 0 0 0 </pose>

File: description/lidar.xacro (robot description, xacro)
@@ -4,12 +4,11 @@
         <parent link="chassis"/>
         <child link="laser_frame"/>
-        <origin xyz="0.1 0 0.07" rpy="0 0 0"/>
+        <origin xyz="0.1 0 0.135" rpy="0 0 0"/>
     </joint>
     <link name="laser_frame">
         <visual>
-            <origin xyz="0.07 -0.24 -0.065" rpy="0 0 -${pi/2}"/>
             <geometry>
-                <!-- <cylinder radius="0.05" length="0.04"/> -->
-                <mesh filename="file://$(find slam_bot)/meshes/Rplidar.stl" scale="0.001 0.001 0.001" />
+                <!-- <mesh filename="file://$(find slam_bot)/meshes/Rplidar.stl" scale="0.001 0.001 0.001" /> -->
+                <mesh filename="package://slam_bot/meshes/Rplidar.stl" scale="0.001 0.001 0.001" />
             </geometry>
             <material name="black"/>
@@ -17,6 +16,6 @@
         <collision>
             <geometry>
-                <!-- <cylinder radius="0.05" length="0.04"/> -->
-                <mesh filename="file://$(find slam_bot)/meshes/Rplidar.stl" scale="0.001 0.001 0.001" />
+                <!-- <mesh filename="file://$(find slam_bot)/meshes/Rplidar.stl" scale="0.001 0.001 0.001" /> -->
+                <mesh filename="package://slam_bot/meshes/Rplidar.stl" scale="0.001 0.001 0.001" />
             </geometry>
         </collision>
@@ -46,5 +45,5 @@
             <plugin name="laser_controller" filename="libgazebo_ros_ray_sensor.so">
                 <ros>
-                    <argument>~/out:=scan</argument>
+                    <remapping>~/out:=scan</remapping>
                 </ros>
                 <output_type>sensor_msgs/LaserScan</output_type>

File: description/robot.urdf.xacro (robot description, xacro)
@@ -11,5 +11,5 @@
     </xacro:unless>
     <xacro:include filename="lidar.xacro" />
-    <xacro:include filename="camera.xacro" />
+    <!-- <xacro:include filename="camera.xacro" /> -->
     <!-- <xacro:include filename="depth_camera.xacro" /> -->
 </robot>

File: description/robot_core.xacro (robot description, xacro)
@@ -3,8 +3,14 @@
     <xacro:include filename="inertial_macros.xacro"/>
     <material name="white">
-        <color rgba="1 1 1 1" />
+        <color rgba="1 1 1 1"/>
+    </material>
+    <material name="black">
+        <color rgba="0 0 0 1"/>
     </material>
     <material name="orange">
         <color rgba="1 0.3 0.1 1"/>
+    </material>
+    <material name="green">
+        <color rgba="0 1 0 1"/>
     </material>
     <material name="yellow">
@@ -13,7 +19,4 @@
     <material name="blue">
         <color rgba="0.2 0.2 1 1"/>
-    </material>
-    <material name="black">
-        <color rgba="0 0 0 1"/>
     </material>
     <material name="red">
@@ -35,5 +38,5 @@
         <parent link="base_link"/>
         <child link="chassis"/>
-        <origin xyz="-0.08 0 0"/>
+        <origin xyz="-0.05 0 0"/>
     </joint>
     <link name="chassis">
@@ -41,5 +44,6 @@
             <origin xyz="0.08 0 0"/>
             <geometry>
-                <mesh filename="file://$(find slam_bot)/meshes/Chassis.stl" scale="0.001 0.001 0.001" />
+                <mesh filename="package://slam_bot/meshes/Chassis.stl" scale="0.001 0.001 0.001" />
+                <!-- <mesh filename="file://$(find slam_bot)/meshes/Chassis.stl" scale="0.001 0.001 0.001" /> -->
                 <!-- <mesh filename="$(find slam_bot)/stl/Chassis.stl" scale="0.001 0.001 0.001" /> -->
             </geometry>

File: description/ros2_control.xacro (robot description, xacro)
@@ -8,8 +8,9 @@
                 <param name="right_wheel_name">right_wheel_joint</param>
                 <param name="loop_rate">30</param>
-                <param name="device">/dev/serial/by-path/pci-0000:03:00.0-usb-0:2:1.0-port0</param>
+                <!-- <param name="device">/dev/serial/by-path/platform-fd500000.pcie-pci-0000:01:00.0-usb-0:1.2:1.0-port0</param> -->
+                <param name="device">/dev/ttyUSB0</param>
                 <param name="baud_rate">57600</param>
                 <param name="timeout_ms">1000</param>
-                <param name="enc_counts_per_rev">3436</param>
+                <param name="enc_counts_per_rev">898</param>
             </hardware>
             <joint name="left_wheel_joint">
